File: kicad/sintez2.kicad_pcb (KiCad board)
At the start: 2 copper layers, 337 x 320 mm, 85 parts, among them X1 JoyL, X2 JoyR, X3 Kbd, X4 DiskDO, X5 Tape, X6 DiskAA

Commit message: T8: re-seed PCB from the updated netlist (arbitration wired, 173 nets)
kinet2pcb re-run after the arbitration/counter wiring; 85 footprints placed (9x10
grid) + Edge.Cuts outline. DSN re-exported for routing.
Connections:
- net H5 renamed S0
- net H6 renamed S1
- net H7 renamed S2
- net ~WE renamed ~WR
- D19 pad 3: H4 -> F
- D2 pad 2: H1 -> H2
- D2 pad 3: H0 -> H1
- D2 pad 6: H2 -> H3
- D2 pad 7: H3 -> H4
- D23 pad 1: (no net) -> ARB_OE0
- D23 pad 10: (no net) -> A1
- D23 pad 11: (no net) -> A5
- D23 pad 12: (no net) -> H1
- D23 pad 13: (no net) -> V3
- D23 pad 14: ARB_CPUVID -> ARB_SELA
- D23 pad 15: (no net) -> GND
- D23 pad 2: ARB_ROWCOL -> ARB_SELB
- D23 pad 3: (no net) -> K10
- D23 pad 4: (no net) -> H0
- D23 pad 5: (no net) -> A10
- D23 pad 6: (no net) -> A0
- D24 pad 1: (no net) -> ARB_OE0
- D24 pad 10: (no net) -> A3
- D24 pad 11: (no net) -> A7
- D24 pad 12: (no net) -> H3
- D24 pad 13: (no net) -> V5
- D24 pad 14: ARB_CPUVID -> ARB_SELA
- D24 pad 15: (no net) -> GND
- D24 pad 2: ARB_ROWCOL -> ARB_SELB
- D24 pad 3: (no net) -> V4
- D24 pad 4: (no net) -> H2
- D24 pad 5: (no net) -> A6
- D24 pad 6: (no net) -> A2
- D25 pad 1: (no net) -> ARB_OE0
- D25 pad 10: (no net) -> A8
- D25 pad 11: (no net) -> A12
- D25 pad 12: (no net) -> K8
- D25 pad 13: (no net) -> K12
- D25 pad 14: ARB_CPUVID -> ARB_SELA
- D25 pad 15: (no net) -> GND
- D25 pad 2: ARB_ROWCOL -> ARB_SELB
- D25 pad 3: (no net) -> K11
- D25 pad 4: (no net) -> H4
- D25 pad 5: (no net) -> A11
- D25 pad 6: (no net) -> A4
- D26 pad 1: (no net) -> ARB_OE0
- D26 pad 10: (no net) -> A14
- D26 pad 11: (no net) -> A15
- D26 pad 12: (no net) -> a2
- D26 pad 13: (no net) -> GND
- D26 pad 14: (no net) -> ARB_SELA
- D26 pad 15: (no net) -> GND
- D26 pad 2: (no net) -> ARB_SELB
- D26 pad 3: (no net) -> GND
- D26 pad 4: (no net) -> K9
- D26 pad 5: (no net) -> A13
- D26 pad 6: (no net) -> A9
- D26 pad 7: (no net) -> VA6
- D26 pad 9: (no net) -> VA7
- D38 pad 1: (no net) -> GND
- D45 pad 6: a2 -> a2_1
- D5 pad 1: (no net) -> nS2
- D5 pad 10: (no net) -> V1
- D5 pad 11: (no net) -> V7
- D5 pad 12: (no net) -> K8
- D5 pad 13: (no net) -> V0
- D5 pad 14: (no net) -> V6
- D5 pad 15: (no net) -> GND
- D5 pad 2: (no net) -> a2
- D5 pad 3: (no net) -> V7
- D5 pad 4: (no net) -> K12
- D5 pad 5: (no net) -> a2
- D5 pad 6: (no net) -> V6
- D5 pad 7: (no net) -> K11
- D5 pad 9: (no net) -> K9
- D7 pad 4: (no net) -> nS2
- D7 pad 5: (no net) -> V2
- D7 pad 6: (no net) -> K10
